File: 12V_Power_PWM.sch (KiCad schematic (older format))
At the start: 4 parts, among them J2 Aviation_Conn_3P, Q3 DMN3016LK3

Commit message: Updated Schematic to correct power page
Parts:
- Q3: symbol _Transistors:DMN3016LK3 -> I2CCaseController_Internal-rescue:DMN3016LK3-_Transistors
Changed lines of the file:
@@
 AR Path="/600035CB/5FFF67B2" Ref="J12"  Part="1"
 AR Path="/600035CE/5FFF67B2" Ref="J13"  Part="1"
-F 0 "J2" H 6178 2996 50  0000 L CNN
+F 0 "J13" H 6178 2996 50  0000 L CNN
 F 1 "Aviation_Conn_3P" H 6178 2905 50  0000 L CNN
 F 2 "_Connectors:Aviation_Conn_3P_Edge" H 5850 3300 50  0001 C CNN
@@
 AR Path="/600035CB/5FFF67B8" Ref="#PWR0117"  Part="1"
 AR Path="/600035CE/5FFF67B8" Ref="#PWR0122"  Part="1"
-F 0 "#PWR0101" H 5450 2800 50  0001 C CNN
+F 0 "#PWR0122" H 5450 2800 50  0001 C CNN
 F 1 "GND" H 5455 2877 50  0000 C CNN
 F 2 "" H 5450 3050 50  0001 C CNN
@@
 AR Path="/600035CB/5FFF67BE" Ref="#PWR0118"  Part="1"
 AR Path="/600035CE/5FFF67BE" Ref="#PWR0123"  Part="1"
-F 0 "#PWR0102" H 5400 2700 50  0001 C CNN
+F 0 "#PWR0123" H 5400 2700 50  0001 C CNN
 F 1 "+12V" H 5415 3023 50  0000 C CNN
 F 2 "" H 5400 2850 50  0001 C CNN
@@
 	5400 2850 5450 2850
 $Comp
-L _Transistors:DMN3016LK3 Q?
+L I2CCaseController_Internal-rescue:DMN3016LK3-_Transistors Q?
 U 1 1 5FFF67C7
 P 5100 3650
@@
 AR Path="/600035CB/5FFF67C7" Ref="Q5"  Part="1"
 AR Path="/600035CE/5FFF67C7" Ref="Q6"  Part="1"
-F 0 "Q3" H 5305 3787 50  0000 L CNN
+F 0 "Q6" H 5305 3787 50  0000 L CNN
 F 1 "DMN3016LK3" H 5305 3696 50  0000 L CNN
 F 2 "_TO_SMD:TO-252-2" H 5300 3575 50  0001 L CIN
@@
 AR Path="/600035CB/5FFF67CF" Ref="#PWR0119"  Part="1"
 AR Path="/600035CE/5FFF67CF" Ref="#PWR0124"  Part="1"
-F 0 "#PWR0103" H 5200 3600 50  0001 C CNN
+F 0 "#PWR0124" H 5200 3600 50  0001 C CNN
 F 1 "GND" H 5205 3677 50  0000 C CNN
 F 2 "" H 5200 3850 50  0001 C CNN
@@
 AR Path="/600035CB/5FFF67D7" Ref="R17"  Part="1"
 AR Path="/600035CE/5FFF67D7" Ref="R18"  Part="1"
-F 0 "R15" H 4770 3946 50  0000 L CNN
+F 0 "R18" H 4770 3946 50  0000 L CNN
 F 1 "10K" H 4770 3855 50  0000 L CNN
 F 2 "Resistor_SMD:R_0603_1608Metric" V 4630 3900 50  0001 C CNN
@@
 AR Path="/600035CB/5FFF67DF" Ref="#PWR0120"  Part="1"
 AR Path="/600035CE/5FFF67DF" Ref="#PWR0128"  Part="1"
-F 0 "#PWR0104" H 4700 3800 50  0001 C CNN
+F 0 "#PWR0128" H 4700 3800 50  0001 C CNN
 F 1 "GND" H 4705 3877 50  0000 C CNN
 F 2 "" H 4700 4050 50  0001 C CNN
@@
 AR Path="/600035CB/5FFF67E7" Ref="D5"  Part="1"
 AR Path="/600035CE/5FFF67E7" Ref="D6"  Part="1"
-F 0 "D3" V 6254 3829 50  0000 L CNN
+F 0 "D6" V 6254 3829 50  0000 L CNN
 F 1 "SD15_SOD323" V 6345 3829 50  0000 L CNN
 F 2 "Diode_SMD:D_SOD-323" H 6300 3550 50  0001 C CNN
@@
 AR Path="/600035CB/5FFF67F1" Ref="#PWR0121"  Part="1"
 AR Path="/600035CE/5FFF67F1" Ref="#PWR0129"  Part="1"
-F 0 "#PWR0105" H 6300 3650 50  0001 C CNN
+F 0 "#PWR0129" H 6300 3650 50  0001 C CNN
 F 1 "GND" H 6305 3727 50  0000 C CNN
 F 2 "" H 6300 3900 50  0001 C CNN
